File: Task4/BMS.kicad_pcb (KiCad board)
At the start: 2 copper layers, 78 parts, among them IC1 DW01, IC2 DW01, IC3 DW01, IC4 DW01, IC5 HY2213-BB3A, IC6 HY2213-BB3A, IC7 HY2213-BB3A, IC8 HY2213-BB3A, Q1 MMBT5551L, Q10 MMBT5551L, Q11 AOD472A, Q12 AOD472A, Q13 AOD472A, Q14 AOD472A, Q15 AOD472A, Q16 AOD472A, Q17 AOD472A, Q18 AOD472A, Q19 AOD472A, Q2 PMST5401, Q20 AOD472A, Q21 MMBT5551L, Q22 BSF030NE2LQ, Q23 BSF030NE2LQ, Q24 BSF030NE2LQ, Q25 BSF030NE2LQ, Q3 PMST5401, Q4 PMST5401, Q5 PMST5401, Q6 PMST5401, Q7 PMST5401, Q8 PMST5401, Q9 PMST5401

Commit message: new design
Parts:
- removed IC1, IC2, IC3, IC4: DW01, DW01:SOT95P280X135-6N
- removed IC5, IC6, IC7, IC8: HY2213-BB3A, HY2213-BB3A:SOT95P280X140-6N
- removed Q11, Q12, Q13, Q14, Q15, Q16, Q17, Q18, Q19, Q20: AOD472A, AOD472A:AOD472A
- removed Q2, Q3, Q4, Q5, Q6, Q7, Q8, Q9: PMST5401, PMST5401:SOT65P210X110-3N
- moved D1 39.1 mm to (122.7, 82.4)
- moved R19 35.5 mm to (107.5, 60.2)
- moved R20 35.5 mm to (107.5, 63.1)
- moved R21 35.5 mm to (107.5, 66.1)
- moved R22 35.5 mm to (107.5, 69.0)
- moved R23 35.5 mm to (107.5, 72.0)
- moved R24 35.5 mm to (107.5, 74.9)
- moved R25 35.5 mm to (107.5, 77.9)
- moved R26 35.5 mm to (107.5, 80.8)
- moved R27 35.5 mm to (107.5, 83.8)
- moved R28 35.5 mm to (111.9, 60.2)
- moved R29 35.5 mm to (111.9, 63.1)
- moved R30 35.5 mm to (111.9, 66.1)
- moved R31 35.5 mm to (111.9, 69.0)
- moved R32 35.5 mm to (111.9, 72.0)
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Routing:
- net Net-(BT4--): track 118.9 -> 0.00 mm, vias 5 -> 8
- net Net-(Q11-D): track 118.1 -> 0.00 mm, vias 0 -> 1
- net Net-(Q1-E): track 100.1 -> 0.00 mm, vias 6 -> 4
- net Net-(Q1-B): track 87.8 -> 0.00 mm, vias 2 -> 3
- net Net-(Q8-B): track 76.2 -> 0.00 mm, vias 2 -> 1
- net Net-(BT2--): track 68.8 -> 0.00 mm, vias 1 -> 6
- net Net-(IC2-OC): track 56.6 -> 0.00 mm, vias 0 -> 1
- net Net-(IC8-VDD): track 55.3 -> 0.00 mm, vias 3 -> 2
- net Net-(IC7-VDD): track 54.4 -> 0.00 mm
- net Net-(Q16-S): track 47.7 -> 0.00 mm, vias 1 -> 3
- net Net-(Q16-G): track 44.8 -> 0.00 mm, vias 2 -> 3
- net Net-(IC4-OC): track 32.4 -> 0.00 mm, vias 0 -> 1
- net Net-(IC6-VDD): track 31.5 -> 0.00 mm, vias 1 -> 2
- net Net-(Q23-D): track 29.8 -> 0.00 mm, vias 0 -> 5
- net Net-(Q24-D): track 28.2 -> 0.00 mm, vias 0 -> 5
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